Commit message: [Modify] Separate mikata_arm_description pkg from bringup pkg.

File: mikata_arm_description/urdf/mikata_arm_4.urdf (robot description, URDF)
Before this commit: robot mikata_arm_4, 8 links, 7 joints
Links:
- link base_link: geometry collision mesh filename=package://mikata_arm_description/meshes/mikata_arm_4_joint1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; visual mesh filename=package://mikata_arm_description/meshes/mikata_arm_4_joint1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
- link left_gripper: geometry collision mesh filename=package://mikata_arm_description/meshes/mikata_arm_4_grippe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; visual mesh filename=package://mikata_arm_description/meshes/mikata_arm_4_grippe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
- link link_2: geometry collision mesh filename=package://mikata_arm_description/meshes/mikata_arm_4_joint2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; visual mesh filename=package://mikata_arm_description/meshes/mikata_arm_4_joint2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
- link link_3: geometry collision mesh filename=package://mikata_arm_description/meshes/mikata_arm_4_joint3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; visual mesh filename=package://mikata_arm_description/meshes/mikata_arm_4_joint3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
- link link_4: geometry collision mesh filename=package://mikata_arm_description/meshes/mikata_arm_4_joint4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; visual mesh filename=package://mikata_arm_description/meshes/mikata_arm_4_joint4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
- link link_5: geometry collision mesh filename=package://mikata_arm_description/meshes/mikata_arm_4_joint5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; visual mesh filename=package://mikata_arm_description/meshes/mikata_arm_4_joint5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
- link right_gripper: geometry collision mesh filename=package://mikata_arm_description/meshes/mikata_arm_4_grippe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; visual mesh filename=package://mikata_arm_description/meshes/mikata_arm_4_grippe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
